File: hardware/W5500_PA_PTT_Control/kicad/w5500-esp32.kicad_pcb (KiCad board)
At the start: 4 copper layers, 72 x 115 mm, 26 parts, among them J1 ESP32_DevKitC_Socket_40P_25.4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, J2 DC_IN_13V8, J5 Power, J6 PTT_ON, Q1 2SC1815, Q3 2SC1815, Q5 2SJ334, U1 TA48033S, U2 L7805

Commit message: W5500制御基板: 放熱器の枠を部品位置に合わせ取付穴位置を反映
- 放熱器の枠(Dwgs.User)が旧位置に残っていたのを修正し、TO-220のタブ裏にそろえて中央の足に穴の中心を合わせた
- 放熱器の取付穴(下端から18mm・幅の中央)の印を追加
- 仕様書(日英)に取付穴位置と部品の取付高さを追記、Word/PDFを再生成

Co-Authored-By: Claude Opus 5.5 <noreply@anthropic.com>
Other:
- board text added: "放熱器 Q5 20x20 (M3穴 高さ18)"
- board text added: "放熱器 U1 20x20 (M3穴 高さ18)"
- board text added: "放熱器 U2 20x20 (M3穴 高さ18)"
- board text removed: "放熱器 Q5 20x20"
- board text removed: "放熱器 U1 20x20"
- board text removed: "放熱器 U2 20x20"
Changed lines of the file:
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@@
 	)
 	(gr_rect
-		(start 151.5 110)
-		(end 171.5 130)
-		(stroke
-			(width 0.1)
-			(type default)
-		)
-		(fill no)
-		(layer "Dwgs.User")
-	)
-	(gr_rect
-		(start 151.5 133)
-		(end 171.5 153)
-		(stroke
-			(width 0.1)
-			(type default)
-		)
-		(fill no)
-		(layer "Dwgs.User")
-	)
-	(gr_rect
-		(start 151.5 156)
-		(end 171.5 176)
+		(start 151.2 118.5)
+		(end 171.2 138.5)
+		(stroke
+			(width 0.1)
+			(type default)
+		)
+		(fill no)
+		(layer "Dwgs.User")
+	)
+	(gr_circle
+		(center 151.2 128.5)
+		(end 152.7 128.5)
+		(stroke
+			(width 0.1)
+			(type default)
+		)
+		(fill no)
+		(layer "Dwgs.User")
+	)
+	(gr_rect
+		(start 151.2 140.5)
+		(end 171.2 160.5)
+		(stroke
+			(width 0.1)
+			(type default)
+		)
+		(fill no)
+		(layer "Dwgs.User")
+	)
+	(gr_circle
+		(center 151.2 150.5)
+		(end 152.7 150.5)
+		(stroke
+			(width 0.1)
+			(type default)
+		)
+		(fill no)
+		(layer "Dwgs.User")
+	)
+	(gr_rect
+		(start 151.2 162.5)
+		(end 171.2 182.5)
+		(stroke
+			(width 0.1)
+			(type default)
+		)
+		(fill no)
+		(layer "Dwgs.User")
+	)
+	(gr_circle
+		(center 151.2 172.5)
+		(end 152.7 172.5)
 		(stroke
 			(width 0.1)
@@
 		)
 	)
-	(gr_text "放熱器 U1 20x20"
-		(at 161.5 120 0)
-		(layer "Dwgs.User")
-		(effects
-			(font
-				(size 0.8 0.8)
-				(thickness 0.12)
-			)
-		)
-	)
-	(gr_text "放熱器 U2 20x20"
-		(at 161.5 143 0)
-		(layer "Dwgs.User")
-		(effects
-			(font
-				(size 0.8 0.8)
-				(thickness 0.12)
-			)
-		)
-	)
-	(gr_text "放熱器 Q5 20x20"
-		(at 161.5 166 0)
-		(layer "Dwgs.User")
-		(effects
+	(gr_text "放熱器 U1 20x20 (M3穴 高さ18)"
+		(at 161.2 120.5 0)
+		(layer "Dwgs.User")
+		(effects
+			(font
+				(size 0.8 0.8)
+				(thickness 0.12)
+			)
+		)
+	)
+	(gr_text "放熱器 U2 20x20 (M3穴 高さ18)"
+		(at 161.2 142.5 0)
+		(layer "Dwgs.User")
+		(effects
+			(font
+				(size 0.8 0.8)
+				(thickness 0.12)
+			)
+		)
+	)
+	(gr_text "放熱器 Q5 20x20 (M3穴 高さ18)"
+		(at 161.2 164.5 0)
+		(layer "Dwgs.User")
+		(effects

Commit message: W5500制御基板: 自動配線・12V系統強化・外付けLED/XHコネクタ化と総点検の修正
- 回路図のGND記号の値が空で別ネットになっていたのを修正
- 内層をGND・+12Vの全面ベタにし、12V出力(/Power)を表裏4mmで配線、残りをFreeroutingで自動配線
- Q1/Q3を2.54mmピッチのTO-92に、R8を1/2W抵抗用フットプリントに変更
- D1/D2を外付けにしてJ7/J8で接続、J6/J7/J8をJST XH(B2B-XH-A)に変更
- C2をTA48033Sデータシートどおり33µF、C1/C3を0.33µFに変更
- Q3ベースにプルダウンR13(10k)を追加、J1のGNDピン21〜24・40を接続
- 仕様書・接続一覧(日英)を更新しWord/PDF・回路図PDF/SVGを再生成

Co-Authored-By: Claude Opus 5.5 <noreply@anthropic.com>
Parts:
- removed D1: LED_Red_3mm, LED_THT:LED_D3.0mm
- removed D2: LED_Green_3mm, LED_THT:LED_D3.0mm
- added J7: LED_PWR, Connector_JST:JST_XH_B2B-XH-A_1x02_P2.50mm_Vertical, F.Cu at (127.0, 132.1)
- added J8: LED_12V, Connector_JST:JST_XH_B2B-XH-A_1x02_P2.50mm_Vertical, F.Cu at (69.0, 134.5)
- added R13: 10k, Resistor_THT:R_Axial_DIN0207_L6.3mm_D2.5mm_P5.08mm_Vertical, F.Cu at (68.0, 100.5)
- C1, C3: value 0.1uF -> 0.33uF
- C2: value 0.1uF -> 33uF
- J6: footprint Connector_Wire:SolderWire-0.5sqmm_1x02_P4.6mm_D0.9mm_OD2.1mm -> Connector_JST:JST_XH_B2B-XH-A_1x02_P2.50mm_Vertical
- Q1, Q3: footprint Package_TO_SOT_THT:TO-92_Inline -> Package_TO_SOT_THT:TO-92_Inline_Wide
- R8: footprint Resistor_THT:R_Axial_DIN0207_L6.3mm_D2.5mm_P5.08mm_Vertical -> Resistor_THT:R_Axial_DIN0309_L9.0mm_D3.2mm_P5.08mm_Vertical
- moved A1 64.5 mm to (75.8, 53.4)
- moved C1 64.5 mm to (110.5, 108.0)
- moved C2 64.5 mm to (110.5, 86.0)
- moved C3 64.5 mm to (110.5, 128.3)
- moved J1 64.5 mm to (77.3, 111.7)
- moved Q5 64.5 mm to (112.0, 116.4)
- moved R10 64.5 mm to (71.5, 100.5)
- moved R11 64.5 mm to (71.5, 109.5)
- moved R12 64.5 mm to (68.0, 91.5)
- moved R6 64.5 mm to (68.0, 64.5)
- moved R7 64.5 mm to (68.0, 73.5)
- moved R8 64.5 mm to (68.0, 82.5)
- moved R9 64.5 mm to (71.5, 118.5)
- moved U2 64.5 mm to (112.0, 94.4)
- moved H1 64.5 mm to (67.0, 49.5)
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Connections:
- J1 pad 21: unconnected-(J1-GND-Pad21) -> GND
- J1 pad 22: unconnected-(J1-GND-Pad22) -> GND
- J1 pad 23: unconnected-(J1-GND-Pad23) -> GND
- J1 pad 24: unconnected-(J1-GND-Pad24) -> GND
- J1 pad 40: unconnected-(J1-GND-Pad40) -> GND
- J1 pad 7: <NO NET> -> GND
Routing:
- net Net-(Q1-B): track 0.00 -> 134.8 mm
- net /+3V3_A: track 0.00 -> 113.4 mm
- net /+5v0: track 0.00 -> 109.7 mm, vias 0 -> 1
- net Net-(Q3-B): track 0.00 -> 109.5 mm
- net /Power: track 0.00 -> 109.4 mm, vias 0 -> 1
- net /GPIO21_W5500_RST: track 0.00 -> 107.6 mm
- net Net-(Q1-C): track 0.00 -> 100.1 mm, vias 0 -> 1
- net Net-(A1-SCK): track 0.00 -> 82.7 mm
- net Net-(A1-CS): track 0.00 -> 82.2 mm
- net Net-(J7-Pin_1): track 0.00 -> 77.5 mm
- net Net-(A1-MOSI): track 0.00 -> 76.6 mm, vias 0 -> 1
- net /GPIO26_PA: track 0.00 -> 74.0 mm
- net Net-(A1-MISO): track 0.00 -> 67.7 mm
- net /GPIO27_PTT: track 0.00 -> 67.5 mm
- net Net-(J8-Pin_1): track 0.00 -> 31.5 mm
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- added copper zone on In2.Cu, net +12V
- added copper zone on In1.Cu, net GND
